File: clock.brd (EAGLE design)
At the start: 99 x 114.5 mm, 15 parts, among them IC1 MEGA16-P

Commit message: 1.1
added smd leds and bugfixed a route.
Parts:
- added LED1, LED2, LED3, LED4: (no value), eagle-ltspice:LED_SML0603
- added R3, R4, R5, R7: (no value), resistor:R0603
Connections:
- new net N$15: LED1.A, R3.1
- new net N$18: LED2.A, R4.1
- new net N$27: LED3.A, R5.1
- new net N$28: LED4.A, R7.1
- net GND: now also LED1.C, LED2.C, LED3.C, LED4.C
- net VCC: now also R3.2, R4.2, R5.2, R7.2
Routing:
- net GND: track 230.4 -> 373.9 mm, vias 1 -> 3
- net VCC: track 138.7 -> 231.2 mm, vias 0 -> 2
- net N$18: track 0.00 -> 8.30 mm
- net N$27: track 0.00 -> 7.30 mm
- net N$15: track 0.00 -> 4.10 mm
- net N$28: track 0.00 -> 3.24 mm
- net N$14: track 43.1 -> 44.2 mm
